File: PCB design files/Signal distribution board (controller board)/signal_distribution_board.brd (EAGLE design)
At the start: 100 x 100 mm, 149 parts, among them U1 CD74HC4067SM96, U10 SN74LV00ADGVR, U11 SN74LV00ADGVR, U12 SN74LV00ADGVR, U13 SN74LV00ADGVR, U14 SN74LV00ADGVR, U15 SN74LV00ADGVR, U16 SN74LV00ADGVR, U17 SN74LV00ADGVR, U18 SN74LV00ADGVR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

Commit message: Updated schematic and board
Parts:
- added R67, R68: 2.2k, rcl:R0805
Connections:
- net GND: now also R67.2, R68.1
- net SDO_2: now also R68.2
- net SDO_5: now also R67.1
Routing:
- net SDO_2: track 197.9 -> 204.6 mm
- net SDO_5: track 209.1 -> 213.3 mm
Changed lines of the file:
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@@
 <attribute name="VALUE" x="12.565" y="72.295" size="1.27" layer="27"/>
 </element>
+<element name="R67" library="rcl" library_urn="urn:adsk.eagle:library:334" package="R0805" package3d_urn="urn:adsk.eagle:package:23553/2" value="2.2k" x="32.7" y="27.75" smashed="yes" rot="R90">
+<attribute name="NAME" x="31.43" y="27.115" size="1.27" layer="25" rot="R90"/>
+<attribute name="POPULARITY" value="86" x="32.7" y="27.75" size="1.778" layer="27" rot="R90" display="off"/>
+<attribute name="SPICEPREFIX" value="R" x="32.7" y="27.75" size="1.778" layer="27" rot="R90" display="off"/>
+<attribute name="VALUE" x="35.24" y="27.115" size="1.27" layer="27" rot="R90"/>
+</element>
+<element name="R68" library="rcl" library_urn="urn:adsk.eagle:library:334" package="R0805" package3d_urn="urn:adsk.eagle:package:23553/2" value="2.2k" x="68" y="71.85" smashed="yes" rot="R90">
+<attribute name="NAME" x="66.73" y="71.215" size="1.27" layer="25" rot="R90"/>
+<attribute name="POPULARITY" value="86" x="68" y="71.85" size="1.778" layer="27" rot="R90" display="off"/>
+<attribute name="SPICEPREFIX" value="R" x="68" y="71.85" size="1.778" layer="27" rot="R90" display="off"/>
+<attribute name="VALUE" x="70.54" y="71.215" size="1.27" layer="27" rot="R90"/>
+</element>
 </elements>
 <signals>
@@
 <contactref element="R65" pad="1"/>
 <contactref element="R66" pad="1"/>
+<contactref element="R67" pad="2"/>
+<contactref element="R68" pad="1"/>
 </signal>
 <signal name="I0_B">
@@
 <via x="77.9" y="81.8" extent="1-16" drill="0.35"/>
 <wire x1="77.9" y1="81.8" x2="77.9" y2="77.78" width="0.254" layer="1"/>
-<wire x1="77.9" y1="77.78" x2="74.02" y2="74.1" width="0.254" layer="1"/>
+<wire x1="77.9" y1="77.78" x2="74.113403125" y2="74.1885875" width="0.254" layer="1"/>
 <contactref element="J17" pad="9"/>
 <contactref element="J1" pad="9"/>
+<wire x1="74.113403125" y1="74.1885875" x2="74.02" y2="74.1" width="0.254" layer="1"/>
 <wire x1="18.98" y1="94.39" x2="18.98" y2="96.48" width="0.254" layer="16"/>
 <wire x1="18.98" y1="96.48" x2="19.5" y2="97" width="0.254" layer="16"/>
@@
 <wire x1="96.95" y1="80.55" x2="96.5128" y2="80.1128" width="0.254" layer="1"/>
 <wire x1="96.95" y1="80.55" x2="96.6" y2="80.9" width="0.254" layer="1"/>
+<contactref element="R68" pad="2"/>
+<wire x1="68" y1="72.8" x2="72.724815625" y2="72.8" width="0.254" layer="1"/>
+<wire x1="72.724815625" y1="72.8" x2="74.113403125" y2="74.1885875" width="0.254" layer="1"/>
 </signal>
 <signal name="SCLK_1">
@@
 <wire x1="21.5" y1="3.036" x2="21.5" y2="5.59" width="0.254" layer="16"/>
 <wire x1="21.5" y1="5.59" x2="21.52" y2="5.61" width="0.254" layer="16"/>
+<contactref element="R67" pad="1"/>
+<wire x1="28.52" y1="26.84" x2="32.66" y2="26.84" width="0.254" layer="1"/>
+<wire x1="32.66" y1="26.84" x2="32.7" y2="26.8" width="0.254" layer="1"/>
 </signal>
 <signal name="SCLK_5">
