File: PCB design files/Signal distribution board (controller board)/signal_distribution_board.sch (EAGLE design)
At the start: 149 parts, among them U1 CD74HC4067SM96, U10 SN74LV00ADGVR, U11 SN74LV00ADGVR, U12 SN74LV00ADGVR, U13 SN74LV00ADGVR, U14 SN74LV00ADGVR, U15 SN74LV00ADGVR, U16 SN74LV00ADGVR, U17 SN74LV00ADGVR, U18 SN74LV00ADGVR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

Commit message: Updated schematic and board
Parts:
- added R67, R68: 2.2k, rcl:R-EU_R0805
Connections:
- net GND: now also R67.2, R68.1
- net SDO_2: now also R68.2
- net SDO_5: now also R67.1
Changed lines of the file:
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@@
 <part name="R66" library="rcl" library_urn="urn:adsk.eagle:library:334" deviceset="R-EU_" device="R0603" package3d_urn="urn:adsk.eagle:package:23555/3" value="1k"/>
 <part name="GND43" library="supply1" library_urn="urn:adsk.eagle:library:371" deviceset="GND" device=""/>
+<part name="R67" library="rcl" library_urn="urn:adsk.eagle:library:334" deviceset="R-EU_" device="R0805" package3d_urn="urn:adsk.eagle:package:23553/2" value="2.2k"/>
+<part name="GND44" library="supply1" library_urn="urn:adsk.eagle:library:371" deviceset="GND" device=""/>
+<part name="R68" library="rcl" library_urn="urn:adsk.eagle:library:334" deviceset="R-EU_" device="R0805" package3d_urn="urn:adsk.eagle:package:23553/2" value="2.2k"/>
+<part name="GND45" library="supply1" library_urn="urn:adsk.eagle:library:371" deviceset="GND" device=""/>
 </parts>
 <sheets>
@@
 <attribute name="VALUE" x="-1224.28" y="162.56" size="1.778" layer="96"/>
 </instance>
+<instance part="R67" gate="G$1" x="-1252.22" y="22.86" smashed="yes" rot="R90">
+<attribute name="NAME" x="-1253.7186" y="19.05" size="1.778" layer="95" rot="R90"/>
+<attribute name="VALUE" x="-1248.918" y="19.05" size="1.778" layer="96" rot="R90"/>
+</instance>
+<instance part="GND44" gate="1" x="-1252.22" y="33.02" smashed="yes" rot="R180">
+<attribute name="VALUE" x="-1249.68" y="35.56" size="1.778" layer="96" rot="R180"/>
+</instance>
+<instance part="R68" gate="G$1" x="-1193.8" y="60.96" smashed="yes" rot="R90">
+<attribute name="NAME" x="-1195.2986" y="57.15" size="1.778" layer="95" rot="R90"/>
+<attribute name="VALUE" x="-1190.498" y="57.15" size="1.778" layer="96" rot="R90"/>
+</instance>
+<instance part="GND45" gate="1" x="-1193.8" y="50.8" smashed="yes">
+<attribute name="VALUE" x="-1196.34" y="48.26" size="1.778" layer="96"/>
+</instance>
 </instances>
 <busses>
@@
 <junction x="-1221.74" y="177.8"/>
 </segment>
+<segment>
+<pinref part="R67" gate="G$1" pin="2"/>
+<pinref part="GND44" gate="1" pin="GND"/>
+<wire x1="-1252.22" y1="27.94" x2="-1252.22" y2="30.48" width="0.1524" layer="91"/>
+</segment>
+<segment>
+<pinref part="R68" gate="G$1" pin="1"/>
+<pinref part="GND45" gate="1" pin="GND"/>
+<wire x1="-1193.8" y1="55.88" x2="-1193.8" y2="53.34" width="0.1524" layer="91"/>
+</segment>
 </net>
 <net name="I0_B" class="0">
@@
 </segment>
 <segment>
-<wire x1="-1216.66" y1="66.04" x2="-1201.42" y2="66.04" width="0.1524" layer="91"/>
+<wire x1="-1216.66" y1="66.04" x2="-1193.8" y2="66.04" width="0.1524" layer="91"/>
 <label x="-1211.58" y="66.04" size="1.778" layer="95"/>
 <pinref part="CN7" gate="A" pin="6"/>
+<pinref part="R68" gate="G$1" pin="2"/>
 </segment>
 </net>
@@
 </segment>
 <segment>
-<wire x1="-1264.92" y1="12.7" x2="-1249.68" y2="12.7" width="0.1524" layer="91"/>
+<wire x1="-1264.92" y1="12.7" x2="-1252.22" y2="12.7" width="0.1524" layer="91"/>
 <label x="-1257.3" y="12.7" size="1.778" layer="95"/>
 <pinref part="CN9" gate="A" pin="4"/>
+<pinref part="R67" gate="G$1" pin="1"/>
+<wire x1="-1252.22" y1="12.7" x2="-1249.68" y2="12.7" width="0.1524" layer="91"/>
+<wire x1="-1252.22" y1="12.7" x2="-1252.22" y2="17.78" width="0.1524" layer="91"/>
+<junction x="-1252.22" y="12.7"/>
 </segment>
 </net>
